File: ARC210_RevD/ARC210_RevD.kicad_sch (KiCad schematic)
At the start: 25 parts, among them J1 Conn_01x03, J2 Conn_01x03, SW1 SW_Push, SW10 SW_Push, SW11 SW_Push, SW12 SW_Push, SW13 SW_Push, SW14 SW_Push, SW2 SW_Push, SW3 SW_Push, SW4 SW_Push, SW5 SW_Push, SW6 SW_Push, SW7 SW_Push, SW8 SW_Push, SW9 SW_Push, U1 MCP23017x-x-SO

Commit message: Alpha Build
Parts:
- added J3: Conn_01x10, Connector_PinHeader_2.54mm:PinHeader_1x10_P2.54mm_Vertical, symbol Connector_Generic:Conn_01x10
Connections:
- net at A1.13 (GND), A1.18 (GND), A1.23 (GND)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: now also J3.2 (Pin_2)
- net at A1.21 (GPIO16): now also J3.10 (pin_10)
- net at A1.22 (GPIO17): now also J3.9 (Pin_9)
- net at A1.24 (GPIO18): now also J3.8 (Pin_8)
- net at A1.25 (GPIO19): now also J3.7 (Pin_7)
- net at A1.26 (GPIO20): now also J3.6 (Pin_6)
- net at A1.27 (GPIO21): now also J3.5 (Pin_5)
- net at A1.29 (GPIO22): now also J3.4 (Pin_4)
- net at A1.31 (GPIO26_ADC0): now also J3.3 (pin_3)
- net at A1.36 (3V3), J1.1 (3v3), J2.1 (3v3)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: now also J3.1 (Pin_1)
Other:
- moved on the sheet: J1, J2
