File: kicad/ARC210_RevE/ARC210_RevE.kicad_pcb (KiCad board)
At the start: 2 copper layers, 142 x 128.4 mm, 52 parts, among them J3 Conn_01x10, SW1 SW_Push, SW10 SW_Push, SW11 SW_Push, SW12 SW_Push, SW13 SW_Push, SW14 SW_Push, SW15 SW_Rotary_1x8_MP, SW16 SW_Rotary_1x8_MP, SW2 SW_Push, SW3 SW_Push, SW4 SW_Push, SW5 SW_Push, SW6 SW_Push, SW7 SW_Push, SW8 SW_Push, SW9 SW_Push

Commit message: added new pcb revision E
Parts:
- J3: moved to F.Cu
- SW15, SW16: footprint Local:RotarySwitch_P-H397_1P8T -> ARC210:RotarySwitch_P-H397_1P8T
- moved ENC6 97.6 mm to (168.1, 119.4), turned to -90 degrees
- moved J3 71.0 mm to (150.0, 73.9), turned to -90 degrees
- moved ENC1 64.6 mm to (242.1, 55.5), turned to 180 degrees
- moved ENC5 49.0 mm to (190.4, 142.4), turned to 0 degrees
- moved ENC7 48.8 mm to (147.1, 119.4), turned to -90 degrees
- moved A1_PICO1 23.0 mm to (186.7, 94.5), turned to 90 degrees
- moved ENC4 22.2 mm to (190.3, 119.5)
- moved ENC2 21.5 mm to (233.1, 119.4)
- moved ENC3 21.3 mm to (211.6, 119.3)
- moved A2_MCP1 9.84 mm to (164.7, 57.2)
- moved C1 9.84 mm to (173.0, 59.8)
- moved R15 9.84 mm to (161.0, 77.2)
- moved R16 9.84 mm to (164.6, 77.1)
- moved R17 9.84 mm to (172.0, 71.5)
- moved R18 9.84 mm to (154.5, 64.2)
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- renumbered REF** to REF_1**, REF** to REF_2**, REF** to REF_3**, REF** to REF_4**
Routing:
- net Net-(A1_PICO1-GPIO1): track 0.00 -> 110.0 mm
- net Net-(A1_PICO1-GPIO0): track 0.00 -> 95.6 mm
- net Net-(A1_PICO1-3V3): track 91.9 -> 9.64 mm
- net Net-(A1_PICO1-GPIO11): track 0.00 -> 43.8 mm
- net Net-(A1_PICO1-GPIO10): track 0.00 -> 37.8 mm
- net Net-(A1_PICO1-GPIO2): track 0.00 -> 35.6 mm
- net Net-(A1_PICO1-GPIO3): track 0.00 -> 33.1 mm
- net Net-(A2_MCP1-V_{SS}): track 553.5 -> 521.5 mm
- net Net-(A1_PICO1-GPIO6): track 0.00 -> 26.8 mm
- net Net-(A1_PICO1-GPIO7): track 0.00 -> 24.3 mm
- net Net-(A1_PICO1-GPIO15): track 0.00 -> 21.2 mm
- net Net-(A1_PICO1-GPIO14): track 0.00 -> 18.8 mm
- net Net-(A1_PICO1-GPIO5): track 26.4 -> 10.8 mm
- net Net-(A1_PICO1-GPIO8): track 0.00 -> 10.9 mm
- net Net-(A1_PICO1-GPIO9): track 0.00 -> 9.85 mm
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Other:
- outline, holes or cut-outs redrawn
