File: kicad/ARC210_RevE/ARC210_RevE.kicad_sch (KiCad schematic)
At the start: 48 parts, among them J3 Conn_01x10, SW1 SW_Push, SW10 SW_Push, SW11 SW_Push, SW12 SW_Push, SW13 SW_Push, SW14 SW_Push, SW15 SW_Rotary_1x8_MP, SW16 SW_Rotary_1x8_MP, SW2 SW_Push, SW3 SW_Push, SW4 SW_Push, SW5 SW_Push, SW6 SW_Push, SW7 SW_Push, SW8 SW_Push, SW9 SW_Push

Commit message: added new pcb revision E
Parts:
- SW15, SW16: footprint Local:RotarySwitch_P-H397_1P8T -> ARC210:RotarySwitch_P-H397_1P8T
Other:
- moved on the sheet: R19, R20
Changed lines of the file:
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@@
 	)
 	(junction
-		(at 187.96 101.6)
-		(diameter 0)
-		(color 0 0 0 0)
-	)
-	(junction
 		(at 194.31 123.19)
 		(diameter 0)
@@
 	)
 	(junction
-		(at 187.96 105.41)
-		(diameter 0)
-		(color 0 0 0 0)
-	)
-	(junction
 		(at 264.16 71.12)
 		(diameter 0)
@@
 	)
 	(junction
+		(at 187.96 100.33)
+		(diameter 0)
+		(color 0 0 0 0)
+	)
+	(junction
+		(at 187.96 105.41)
+		(diameter 0)
+		(color 0 0 0 0)
+	)
+	(junction
 		(at 264.16 139.7)
 		(diameter 0)
@@
 	(wire
 		(pts
-			(xy 198.12 109.22) (xy 195.58 109.22)
+			(xy 198.12 110.49) (xy 195.58 110.49)
 		)
 		(stroke
@@
 	(wire
 		(pts
-			(xy 198.12 107.95) (xy 198.12 109.22)
+			(xy 198.12 107.95) (xy 198.12 110.49)
 		)
 		(stroke
@@
 	(wire
 		(pts
+			(xy 187.96 100.33) (xy 187.96 105.41)
+		)
+		(stroke
+			(width 0)
+			(type default)
+		)
+	)
+	(wire
+		(pts
 			(xy 46.99 149.86) (xy 78.74 149.86)
 		)
@@
 	(wire
 		(pts
-			(xy 187.96 101.6) (xy 187.96 105.41)
-		)
-		(stroke
-			(width 0)
-			(type default)
-		)
-	)
-	(wire
-		(pts
 			(xy 129.54 76.2) (xy 140.97 76.2)
 		)
@@
 	(wire
 		(pts
-			(xy 198.12 102.87) (xy 198.12 101.6)
+			(xy 198.12 102.87) (xy 198.12 100.33)
 		)
 		(stroke
@@
 	(wire
 		(pts
-			(xy 198.12 101.6) (xy 195.58 101.6)
+			(xy 198.12 100.33) (xy 195.58 100.33)
 		)
 		(stroke
@@
 	(wire
 		(pts
+			(xy 187.96 49.53) (xy 187.96 100.33)
+		)
+		(stroke
+			(width 0)
+			(type default)
+		)
+	)
+	(wire
+		(pts
 			(xy 261.62 105.41) (xy 264.16 105.41)
 		)
@@
 	(wire
 		(pts
-			(xy 187.96 105.41) (xy 187.96 109.22)
+			(xy 187.96 105.41) (xy 187.96 110.49)
 		)
 		(stroke
@@
 	(wire
 		(pts
-			(xy 187.96 49.53) (xy 187.96 101.6)
-		)
-		(stroke
-			(width 0)
-			(type default)
-		)
-	)
-	(wire
-		(pts
 			(xy 142.24 33.02) (xy 66.04 33.02)
 		)
@@
 	(symbol
 		(lib_id "Device:R")
-		(at 191.77 109.22 270)
+		(at 191.77 110.49 270)
 		(unit 1)
 		(body_style 1)
@@
 		(fields_autoplaced yes)
 		(property "Reference" "R20"
-			(at 191.77 102.87 90)
+			(at 191.77 104.14 90)
 			(show_name no)
 			(do_not_autoplace no)
@@
 		)
 		(property "Value" "10K"
-			(at 191.77 105.41 90)
+			(at 191.77 106.68 90)
 			(show_name no)
 			(do_not_autoplace no)
@@
 		)
 		(property "Footprint" "Resistor_SMD:R_0805_2012Metric_Pad1.20x1.40mm_HandSolder"
-			(at 191.77 107.442 90)
+			(at 191.77 108.712 90)
 			(hide yes)
 			(show_name no)
@@
 		)
 		(property "Datasheet" ""
-			(at 191.77 109.22 0)
+			(at 191.77 110.49 0)
 			(hide yes)
 			(show_name no)
@@
 		)
 		(property "Description" "Resistor"
-			(at 191.77 109.22 0)
+			(at 191.77 110.49 0)
 			(hide yes)
 			(show_name no)
@@
 			)
 		)
-		(property "Footprint" "Local:RotarySwitch_P-H397_1P8T"
+		(property "Footprint" "ARC210:RotarySwitch_P-H397_1P8T"
 			(at 110.49 -40.64 0)
 			(hide yes)
@@
 			)
 		)
-		(property "Footprint" "Local:RotarySwitch_P-H397_1P8T"
+		(property "Footprint" "ARC210:RotarySwitch_P-H397_1P8T"
 			(at 194.31 -41.91 0)
 			(hide yes)
@@
 	(symbol
 		(lib_id "Device:R")
-		(at 191.77 101.6 270)
+		(at 191.77 100.33 270)
 		(unit 1)
 		(body_style 1)
@@
 		(fields_autoplaced yes)
 		(property "Reference" "R19"
-			(at 191.77 95.25 90)
+			(at 191.77 93.98 90)
 			(show_name no)
 			(do_not_autoplace no)
@@
 		)
 		(property "Value" "10K"
-			(at 191.77 97.79 90)
+			(at 191.77 96.52 90)
 			(show_name no)
 			(do_not_autoplace no)
@@
 		)
 		(property "Footprint" "Resistor_SMD:R_0805_2012Metric_Pad1.20x1.40mm_HandSolder"
-			(at 191.77 99.822 90)
+			(at 191.77 98.552 90)
 			(hide yes)
 			(show_name no)
@@
 		)
 		(property "Datasheet" ""
-			(at 191.77 101.6 0)
+			(at 191.77 100.33 0)
 			(hide yes)
 			(show_name no)
@@
 		)
 		(property "Description" "Resistor"
-			(at 191.77 101.6 0)
+			(at 191.77 100.33 0)
 			(hide yes)
 			(show_name no)
